File: MagicController.kicad_sch (KiCad schematic)
At the start: 28 parts, among them SW1 TS-1187A-B-A-B, SW2 TS-1187A-B-A-B, U1 CH340C_C7464026, U2 AMS1117-3.3, U3 ESP32-WROOM-32E(8MB), U4 ESP32-S3-WROOM-1, U5 DS18B20U, U6 CH224K

Commit message: easyeda2kidad from csv
añadido script para cargar las libs
Parts:
- removed C1: 0.1u, easyeda2kicad:C0603, symbol easyeda2kicad:CC0603KRX7R9BB104
- removed R1, R2: 5k1, easyeda2kicad:R0603, symbol easyeda2kicad:0603WAF5101T5E
- removed U1: CH340C_C7464026, easyeda2kicad:SOP-16_L10.0-W3.9-P1.27-LS6.0-BL, symbol easyeda2kicad:CH340C_C7464026
- removed U3: ESP32-WROOM-32E(8MB), easyeda2kicad:WIFI-SMD_ESP32-WROOM-32E, symbol easyeda2kicad:ESP32-WROOM-32E(8MB)
- removed USBC1: TYPE-C-31-M-12, easyeda2kicad:USB-C_SMD-TYPE-C-31-M-12, symbol easyeda2kicad:TYPE-C-31-M-12
Other:
- note removed: "ESP32"
- note removed: "USB Connector"
- note removed: "USB-UART Bridge"
- moved on the sheet: C2, C3, C4, LED1, LED2, R10, R11, R12, R3, R4, R5, R6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
