File: boilerplate/esp32/esp32_boilerplate.kicad_pcb (KiCad board)
At the start: 2 copper layers, 100 x 100 mm, 15 parts, among them SW1 TS-1187A-B-A-B, SW2 TS-1187A-B-A-B, U1 CH340C_C7464026, U2 AMS1117-3.3, U3 ESP32-WROOM-32E(8MB)

Commit message: Minors
Parts:
- moved U3 65.7 mm to (92.7, 63.5), turned to 0 degrees
- moved SW1 37.2 mm to (109.8, 56.1)
- moved SW2 27.0 mm to (109.8, 62.6)
- moved C3 19.1 mm to (132.3, 69.6), turned to 0 degrees
- moved C2 18.6 mm to (132.3, 57.6), turned to 0 degrees
- moved R3 17.6 mm to (107.8, 69.1), turned to 0 degrees
- moved LED1 15.8 mm to (107.8, 71.6), turned to 180 degrees
- moved U2 14.0 mm to (132.3, 63.6), turned to 90 degrees
- moved LED2 13.8 mm to (111.5, 69.1), turned to 180 degrees
- moved R7 11.1 mm to (111.6, 71.7), turned to 0 degrees
- moved U1 7.27 mm to (122.1, 67.3)
- moved R2 7.10 mm to (124.8, 61.0)
- moved C1 6.95 mm to (117.0, 70.9)
- moved R1 6.87 mm to (119.2, 61.0)
- moved USBC1 6.76 mm to (122.3, 56.7)
Routing:
- net /3V3: track 0.00 -> 11.7 mm
- net /5V: track 0.00 -> 3.51 mm
- net Net-(USBC1-CC1): track 0.00 -> 2.11 mm
- net Net-(USBC1-CC2): track 0.00 -> 2.11 mm
